File: power-supply.sch (KiCad schematic (older format))
At the start: 122 parts, among them Q10 2N7002, Q11 2N7002, Q12 2N7002, Q13 2N7002, Q14 2N7002, Q15 2N7002, Q16 2N7002, Q4 IRLML6402TRPBF, Q5 IRLML6402TRPBF, Q6 IRLML6402TRPBF, Q7 IRLML6402TRPBF, Q8 IRLML6402TRPBF, Q9 IRLML6402TRPBF, U13 LM21212-2, U14 SN74LVC1G11DBVR, U15 SN74LS08DBR, U16 TPS62823DLCT

Commit message: Component cleanup
Parts:
- C100, C?: footprint ecp5-dc-scm-footprints:0402-cap -> fmc2sata-footprints:0402-cap; symbol ecp5-dc-scm:C_100n_0402 -> fmc2sata:C_100n_0402
- C106: footprint ecp5-dc-scm-footprints:0402-cap -> fmc2sata-footprints:0402-cap; symbol ecp5-dc-scm:C_1n8_0402 -> fmc2sata:C_1n8_0402
- C107: footprint ecp5-dc-scm-footprints:0402-cap -> fmc2sata-footprints:0402-cap; symbol ecp5-dc-scm:C_180p_0402 -> fmc2sata:C_180p_0402
- C108: footprint ecp5-dc-scm-footprints:0402-res -> fmc2sata-footprints:0402-res; symbol ecp5-dc-scm:C_750p_0402 -> fmc2sata:C_750p_0402
- C113, C127, C132, C? (x12): footprint ecp5-dc-scm-footprints:0402-cap -> fmc2sata-footprints:0402-cap; symbol ecp5-dc-scm:C_10u_0402 -> fmc2sata:C_10u_0402
- C122, C? (x4): footprint ecp5-dc-scm-footprints:0402-res -> fmc2sata-footprints:0402-res; symbol ecp5-dc-scm:C_120p_0402 -> fmc2sata:C_120p_0402
- C? (x3): footprint ecp5-dc-scm-footprints:0603_25V-res -> fmc2sata-footprints:0603_25V-res; symbol ecp5-dc-scm:C_2u2_0603_25V -> fmc2sata:C_2u2_0603_25V
- C? (x2): footprint ecp5-dc-scm-footprints:0402-cap -> fmc2sata-footprints:0402-cap; symbol ecp5-dc-scm:C_10n_0402 -> fmc2sata:C_10n_0402
- C?: footprint ecp5-dc-scm-footprints:0402-cap -> fmc2sata-footprints:0402-cap; symbol ecp5-dc-scm:C_4n7_0402 -> fmc2sata:C_4n7_0402
- C?: footprint ecp5-dc-scm-footprints:0402-cap -> fmc2sata-footprints:0402-cap; symbol ecp5-dc-scm:C_47p_0402 -> fmc2sata:C_47p_0402
- C?: footprint ecp5-dc-scm-footprints:1210-cap -> fmc2sata-footprints:1210-cap; symbol ecp5-dc-scm:C_47u_1210 -> fmc2sata:C_47u_1210
- C? (x2): footprint ecp5-dc-scm-footprints:0805-cap -> fmc2sata-footprints:0805-cap; symbol ecp5-dc-scm:C_10u_0805 -> fmc2sata:C_10u_0805
- C? (x3): footprint ecp5-dc-scm-footprints:0603-cap -> fmc2sata-footprints:0603-cap; symbol ecp5-dc-scm:C_47u_0603 -> fmc2sata:C_47u_0603
- D10, D11, D12, D13, D7, D8, D9: footprint ecp5-dc-scm-footprints:LED_0603 -> fmc2sata-footprints:LED_0603; symbol ecp5-dc-scm:LG_L29K-G2J1-24-Z -> fmc2sata:LG_L29K-G2J1-24-Z
- D?: footprint ecp5-dc-scm-footprints:PDS760-13 -> fmc2sata-footprints:PDS760-13; symbol ecp5-dc-scm:PDS760-13 -> fmc2sata:PDS760-13
- F?: footprint ecp5-dc-scm-footprints:1206-Fuse-Littelfuse-0466-0-0-MFG -> fmc2sata-footprints:1206-Fuse-Littelfuse-0466-0-0-MFG; symbol ecp5-dc-scm:0466003.NR -> fmc2sata:0466003.NR
- IC?: footprint ecp5-dc-scm-footprints:WSON-10_4x4 -> fmc2sata-footprints:WSON-10_4x4; symbol ecp5-dc-scm:TPS54561 -> fmc2sata:TPS54561
- J?: footprint ecp5-dc-scm-footprints:PinHeader_1x2_P2mm_Drill1mm_RA -> fmc2sata-footprints:PinHeader_1x2_P2mm_Drill1mm_RA; symbol ecp5-dc-scm:S2B-PH-K-S_LF__SN_ -> fmc2sata:S2B-PH-K-S_LF__SN_
- L1: footprint ecp5-dc-scm-footprints:Coilcraft-XAL5030 -> fmc2sata-footprints:Coilcraft-XAL5030; symbol ecp5-dc-scm:XAL5030-801 -> fmc2sata:XAL5030-801
- L7, L? (x4): footprint ecp5-dc-scm-footprints:IHLP-1212AE -> fmc2sata-footprints:IHLP-1212AE; symbol ecp5-dc-scm:IHLP1212AEERR47M11 -> fmc2sata:IHLP1212AEERR47M11
- L?: footprint ecp5-dc-scm-footprints:WE_7447798720 -> fmc2sata-footprints:WE_7447798720; symbol ecp5-dc-scm:WE_7447798720 -> fmc2sata:WE_7447798720
- Q10, Q11, Q12, Q13, Q14, Q15, Q16: footprint ecp5-dc-scm-footprints:SOT-23-3 -> fmc2sata-footprints:SOT-23-3; symbol ecp5-dc-scm:2N7002 -> fmc2sata:2N7002
- Q4, Q5, Q6, Q7, Q8, Q9: footprint ecp5-dc-scm-footprints:SOT-23-3 -> fmc2sata-footprints:SOT-23-3; symbol ecp5-dc-scm:IRLML6402TRPBF -> fmc2sata:IRLML6402TRPBF
- R100, R101, R102, R103, R104, R105, R106, R98: footprint ecp5-dc-scm-footprints:0402-res -> fmc2sata-footprints:0402-res; symbol ecp5-dc-scm:R_10k_0402 -> fmc2sata:R_10k_0402
- R107, R108, R109, R110, R111, R112, R113, R? (x3): footprint ecp5-dc-scm-footprints:0402-res -> fmc2sata-footprints:0402-res; symbol ecp5-dc-scm:R_1k_0402 -> fmc2sata:R_1k_0402
- R122, R?: footprint ecp5-dc-scm-footprints:0402-res -> fmc2sata-footprints:0402-res; symbol ecp5-dc-scm:R_453k_0402 -> fmc2sata:R_453k_0402
- R123, R? (x5): footprint ecp5-dc-scm-footprints:0402-res -> fmc2sata-footprints:0402-res; symbol ecp5-dc-scm:R_100k_0402 -> fmc2sata:R_100k_0402
- R88: footprint ecp5-dc-scm-footprints:0603-res -> fmc2sata-footprints:0603-res; symbol ecp5-dc-scm:R_10R_0603 -> fmc2sata:R_10R_0603
- R89: footprint ecp5-dc-scm-footprints:0402-res -> fmc2sata-footprints:0402-res; symbol ecp5-dc-scm:R_47k_0402 -> fmc2sata:R_47k_0402
- R93: footprint ecp5-dc-scm-footprints:0402-res -> fmc2sata-footprints:0402-res; symbol ecp5-dc-scm:R_4k7_0402 -> fmc2sata:R_4k7_0402
- R99: footprint ecp5-dc-scm-footprints:0402-res -> fmc2sata-footprints:0402-res; symbol ecp5-dc-scm:R_470k_0402 -> fmc2sata:R_470k_0402
- R?: footprint ecp5-dc-scm-footprints:0402-res -> fmc2sata-footprints:0402-res; symbol ecp5-dc-scm:R_1k1_0402 -> fmc2sata:R_1k1_0402
- R?: footprint ecp5-dc-scm-footprints:1206-res -> fmc2sata-footprints:1206-res; symbol ecp5-dc-scm:R_0R_1206 -> fmc2sata:R_0R_1206
- R?: footprint ecp5-dc-scm-footprints:0402-res -> fmc2sata-footprints:0402-res; symbol ecp5-dc-scm:R_243k_0402 -> fmc2sata:R_243k_0402
- R?: footprint ecp5-dc-scm-footprints:0402-res -> fmc2sata-footprints:0402-res; symbol ecp5-dc-scm:R_16k9_0402 -> fmc2sata:R_16k9_0402
- R?: footprint ecp5-dc-scm-footprints:0402-res -> fmc2sata-footprints:0402-res; symbol ecp5-dc-scm:R_10k2_0402 -> fmc2sata:R_10k2_0402
- R?: footprint ecp5-dc-scm-footprints:0402-res -> fmc2sata-footprints:0402-res; symbol ecp5-dc-scm:R_49R9_0402 -> fmc2sata:R_49R9_0402
- R?: footprint ecp5-dc-scm-footprints:0402-res -> fmc2sata-footprints:0402-res; symbol ecp5-dc-scm:R_53k6_0402 -> fmc2sata:R_53k6_0402
- R?: footprint ecp5-dc-scm-footprints:0402-res -> fmc2sata-footprints:0402-res; symbol ecp5-dc-scm:R_200k_0402 -> fmc2sata:R_200k_0402
- R?: footprint ecp5-dc-scm-footprints:0402-res -> fmc2sata-footprints:0402-res; symbol ecp5-dc-scm:R_124k_0402 -> fmc2sata:R_124k_0402
- R?: footprint ecp5-dc-scm-footprints:0603-res -> fmc2sata-footprints:0603-res; symbol ecp5-dc-scm:R_66k5_0603 -> fmc2sata:R_66k5_0603
- TP7, TP?: footprint ecp5-dc-scm-footprints:Testpoint_smd_1mm -> fmc2sata-footprints:Testpoint_smd_1mm; symbol ecp5-dc-scm:TP_SMD1MM -> fmc2sata:TP_SMD1MM
- TP? (x2): footprint ecp5-dc-scm-footprints:PROBE_PAD_1206 -> fmc2sata-footprints:PROBE_PAD_1206; symbol ecp5-dc-scm:RCW-0C -> fmc2sata:RCW-0C
- U13: footprint ecp5-dc-scm-footprints:HTSSOP-20_TI-PWP -> fmc2sata-footprints:HTSSOP-20_TI-PWP; symbol ecp5-dc-scm:LM21212-2 -> fmc2sata:LM21212-2
- U14: footprint ecp5-dc-scm-footprints:SOT-23-6 -> fmc2sata-footprints:SOT-23-6; symbol ecp5-dc-scm:SN74LVC1G11DBVR -> fmc2sata:SN74LVC1G11DBVR
- U15: symbol ecp5-dc-scm:SN74LS08DBR -> fmc2sata:SN74LS08DBR
- U16, U? (x4): footprint ecp5-dc-scm-footprints:QFN-8_2x1mm -> fmc2sata-footprints:QFN-8_2x1mm; symbol ecp5-dc-scm:TPS62823DLCT -> fmc2sata:TPS62823DLCT
- U?: footprint ecp5-dc-scm-footprints:VSSOP8-Texas_Instruments-DGK0008A -> fmc2sata-footprints:VSSOP8-Texas_Instruments-DGK0008A; symbol ecp5-dc-scm:LM3881MME_NOPB -> fmc2sata:LM3881MME_NOPB
